File: ESP32.kicad_sch (KiCad schematic)
At the start: 27 parts, among them J8 629105136821, Q1 SS8050-G, Q2 SS8050-G, U1 CP2102N-A02-GQFN28, U2 ESP32-WROOM-32UE

Commit message: R1
ESP32-R1
Parts:
- removed D4: LESD5D5.0CT1G, proj_library:SOD-523, symbol proj_library:LESD5D5.0CT1G
- removed J8: 629105136821, proj_library:629105136821, symbol proj_library:629105136821
- removed R8: 2.00k, proj_library:R0603, symbol proj_library:CRCW06032K00FKEAC
- added D4: LESD5Z5.0T1G, proj_library:SOD-523, symbol proj_library:LESD5Z5.0T1G
- added J2: GSB1CA11101DSHR, proj_library:AMPHENOL_GSB1CA11101DSHR, symbol proj_library:GSB1CA11101DSHR
- added R24, R25: 5.11k, proj_library:R0603, symbol proj_library:CRCW06035K11FKEAC
- added R8: 1.00k, proj_library:R0603, symbol proj_library:CRCW06031K00FKEAC
- C1, C3, C5, C6, C7: MPN (none) -> CC0603KRX7R7BB104; Manufacturer (none) -> YAGEO
- C2: MPN (none) -> CL10A475KP8NNNC; Manufacturer (none) -> Samsung Electro-Mechanics
- C4: MPN (none) -> CL21A226MOCLRNC; Manufacturer (none) -> Samsung Electro-Mechanics
- D1: MPN (none) -> BAT760-7
- D2, D3: MPN (none) -> LESD5D5.0CT1G
- Q1, Q2: MPN (none) -> SS8050-G
- R10, R15, R16, R9: MPN (none) -> CRCW060310K0FKEAC; Manufacturer (none) -> Vishay Dale
- R11: MPN (none) -> CRCW060322K1FKEAC; Manufacturer (none) -> Vishay Dale
- R12: MPN (none) -> CRCW060347K5FKEAC; Manufacturer (none) -> Vishay Dale
- R13, R14: MPN (none) -> CRCW06030000Z0EAC; Manufacturer (none) -> Vishay Dale
- S1, S2: value PTS636_SL50_SMTR_LFS -> PTS636 SL50 SMTR LFS; MPN (none) -> PTS636 SL50 SMTR LFS
- U1: MPN (none) -> CP2102N-A02-GQFN28
- U2: footprint proj_library:ESP32WROOM32UE -> proj_library:ESP32-32UE_EXP; MPN (none) -> ESP32-WROOM-32UE; Manufacturer Espressif -> Espressif Systems
Connections:
- net GND: now also D4.2, J2.A1 (GND_A), J2.A12 (GND_A_1), J2.B1 (GND_B), J2.B12 (GND_B_1), J2.SH1 (SHIELD), J2.SH2 (SHIELD_1), J2.SH3 (SHIELD_2), J2.SH4 (SHIELD_3), R24.2, R25.2
- net P3V3: now also R8.1
- net USB_DN: now also J2.A7 (DN1), J2.B7 (DN2)
- net USB_DP: now also J2.A6 (DP1), J2.B6 (DP2)
- net VBUS: now also D4.1, J2.A4 (VBUS_A), J2.A9 (VBUS_A_1), J2.B4 (VBUS_B), J2.B9 (VBUS_B_1)
- net RST: now reaches U2.23 (IO15)
- net CS2: now reaches U2.24 (IO2)
- net CS3: now reaches U2.26 (IO4)
- net INT: now reaches U2.7 (IO35)
- net at U1.9 (~{RST}): now also R8.2
- net PVESC renamed PVIN
- net V_CLK renamed SCK
- net V_CS renamed CS
- net V_MISO renamed MISO
- net V_MOSI renamed MOSI
- new net CC1: J2.A5 (CC1), R24.1
- new net CC2: J2.B5 (CC2), R25.1
- no-connect marks 27 -> 24
Other:
- note added: "Make this a 10u to fix boot problem"
- moved on the sheet: C6, C7, D1, Q1, Q2, R13, R14, R15, R16, S1, S2
