File: PSU.kicad_sch (KiCad schematic)
At the start: 14 parts, among them U3 AP62201WU-7

Commit message: R1
ESP32-R1
Parts:
- added R26: 0, proj_library:R0603, symbol proj_library:CRCW06030000Z0EAC
- C10: MPN (none) -> CC0603KRX7R7BB104; Manufacturer (none) -> YAGEO
- C11, C12: MPN (none) -> CL21A226MOCLRNC; Manufacturer (none) -> Samsung Electro-Mechanics
- C8: MPN (none) -> CL10B334KO8NNNC; Manufacturer (none) -> Samsung Electro-Mechanics
- C9: MPN (none) -> CL21A106KOQNNNE; Manufacturer (none) -> Samsung Electro-Mechanics
- D5: MPN (none) -> 150060VS75000
- L1: MPN (none) -> LSXNH8080YBL3R3NJG
- R17, R23: MPN (none) -> CRCW06030000Z0EAC; Manufacturer (none) -> Vishay Dale
- R18: MPN (none) -> CRCW0603100KFKEAC; Manufacturer (none) -> Vishay Dale
- R19: MPN (none) -> CRCW060331K6FKEAC; Manufacturer (none) -> Vishay Dale
- R20: MPN (none) -> CRCW0603255RFKEAC; Manufacturer (none) -> Vishay Dale
- R21: MPN (none) -> CRCW060310K0FKEAC; Manufacturer (none) -> Vishay Dale
- U3: MPN (none) -> AP62201WU-7
Connections:
- net at C11.1, C12.1, L1.2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: now also R26.1; no longer R19.1
- new net: R19.1, R26.2
Other:
- moved on the sheet: R19, R21
